File: 2-ECAD/OpenNAS.kicad_sch (KiCad schematic)
At the start: 0 parts

Commit message: power and esp32
Parts:
- added C1: 22uF, symbol Device:C
- added C10, C14, C7, C8: 10u, symbol Device:C
- added C11, C13, C2, C4, C5, C9: 0.1u, symbol Device:C
- added C12, C6: 22p, symbol Device:C
- added C3: 1u, symbol Device:C
- added D1, D2, D3: LESD5D5.0CT1G, symbol 0_Diode:LESD5D5.0CT1G
- added D4, D5: DSS24, symbol 0_Diode:DSS24
- added J1, J2: 470531000, symbol 0_Connector:470531000
- added J3, J4: M5082VK-04P, symbol 0_Connector:M5082VK-04P
- added J5: USB4105, symbol 0_Connector:USB4105
- added J6: 5034802000, symbol 0_Connector:5034802000
- added L1, L2: 2.2u, symbol Device:L
- added R1, R11, R2, R3, R8: 10k, symbol Device:R
- added R10, R13: 150k, symbol Device:R
- added R12, R9: 680k, symbol Device:R
- added R4, R5: 5.1k, symbol Device:R
- added R6, R7: 33R, symbol Device:R
- added SW1: 1825027, symbol 0_Switch:1825027
- added U1: ESP32-C5-WROOM-1-N8R8, symbol 0_MCU_Espressif:ESP32-C5-WROOM-1-N8R8
- added U2, U3: SY8088AAC, symbol 0_Converter_DCDC:SY8088AAC
Connections:
- new net: C6.2, R10.1, R9.2, U2.5 (FB)
- new net: C12.2, R12.2, R13.1, U3.5 (FB)
- new net: D2.1, J5.A7 (Dn1), J5.B7 (Dn2), R6.1
- new net: J5.A5 (CC1), R5.1
- new net: D1.1, J5.A6 (Dp1), J5.B6 (Dp2), R7.1
- new net: J5.B5 (CC2), R4.1
- new net: L1.1, U2.3 (LX)
- new net: R8.2, U2.1 (EN)
- new net: L2.1, U3.3 (LX)
- new net 12V: J1.2 (PWR), J2.2 (PWR), J3.1 (12V), J4.1 (12V)
- new net 3V3: C12.1, C13.1, C14.1, L2.2, R12.1
- new net 5V: D5.2, J3.4 (5V), J4.4 (5V)
- new net EN_PHRL: R11.1, U1.15 (IO28), U3.1 (EN)
- new net FAN_PWM_0: J2.4 (PWM), U1.26 (IO25)
- new net FAN_PWM_1: J1.4 (PWM), U1.18 (IO27)
- new net FAN_TACH_0: J2.3 (RPM), R3.2, U1.23 (IO24)
- new net FAN_TACH_1: J1.3 (RPM), R2.2, U1.27 (IO26)
- new net GND: C1.2, C10.2, C11.2, C13.2, C14.2, C2.2, C3.2, C4.2, C5.2, C7.2, C8.2, C9.2, D1.2, D2.2, D3.2, J1.1 (GND), J2.1 (GND), J3.2 (GND), J3.3 (GND), J4.2 (GND), J4.3 (GND), J5.1 (MP), J5.2 (MP), J5.3 (MP), J5.4 (MP), J5.A1 (GND), J5.A12 (GND), J5.B1 (GND), J5.B12 (GND), R10.2, R11.2, R13.2, R4.2, R5.2, SW1.1 (COM), SW1.3 (MP), SW1.4 (MP), U1.1 (GND), U1.28 (GND), U1.29 (EPAD), U2.2 (GND), U3.2 (GND)
- new net MCU_3V3: C1.1, C2.1, C6.1, C7.1, C9.1, L1.2, R1.1, R2.1, R3.1, R9.1, U1.2 (3V3)
- new net MCU_EN: C3.1, C4.1, R1.2, SW1.2 (NO), U1.3 (EN)
- new net MCU_RX0: U1.24 (RX0)
- new net MCU_TX0: U1.25 (TX0)
- new net MCU_USB_D+: R6.2, U1.14 (IO14)
- new net MCU_USB_D-: R7.2, U1.13 (IO13)
- new net MCU_X_IO0: U1.6 (IO0)
- new net MCU_X_IO1: U1.7 (IO1)
- new net VBUS: D3.1, D4.2, J5.A4 (VBUS), J5.A9 (VBUS), J5.B4 (VBUS), J5.B9 (VBUS)
- new net VCC_5V: C10.1, C11.1, C5.1, C8.1, D4.1, D5.1, R8.1, U2.4 (IN), U3.4 (IN)
- no-connect marks 0 -> 3

Commit message: power done
Parts:
- removed C1: 22uF, symbol Device:C
- removed C10, C14, C7, C8: 10u, symbol Device:C
- removed C11, C13, C2, C4, C5, C9: 0.1u, symbol Device:C
- removed C12, C6: 22p, symbol Device:C
- removed C3: 1u, symbol Device:C
- removed D1, D2, D3: LESD5D5.0CT1G, symbol 0_Diode:LESD5D5.0CT1G
- removed D4, D5: DSS24, symbol 0_Diode:DSS24
- removed J1, J2: 470531000, symbol 0_Connector:470531000
- removed J3, J4: M5082VK-04P, symbol 0_Connector:M5082VK-04P
- removed J5: USB4105, symbol 0_Connector:USB4105
- removed J6: 5034802000, symbol 0_Connector:5034802000
- removed L1, L2: 2.2u, symbol Device:L
- removed R1, R11, R2, R3, R8: 10k, symbol Device:R
- removed R10, R13: 150k, symbol Device:R
- removed R12, R9: 680k, symbol Device:R
- removed R4, R5: 5.1k, symbol Device:R
- removed R6, R7: 33R, symbol Device:R
- removed SW1: 1825027, symbol 0_Switch:1825027
- removed U1: ESP32-C5-WROOM-1-N8R8, symbol 0_MCU_Espressif:ESP32-C5-WROOM-1-N8R8
- removed U2, U3: SY8088AAC, symbol 0_Converter_DCDC:SY8088AAC
Connections:
- no-connect marks 3 -> 0
Other:
- added sheet HDD1 (hdd.kicad_sch)
- added sheet HDD2 (hdd.kicad_sch)
- added sheet HDD3 (hdd.kicad_sch)
- added sheet HDD4 (hdd.kicad_sch)
- added sheet HDD5 (hdd.kicad_sch)
- added sheet HDD6 (hdd.kicad_sch)
- added sheet MCU (mcu.kicad_sch)
- added sheet Power (power.kicad_sch)

Commit message: production version
Other:
- sheet HDD2 ports: added ACT; removed none
- sheet HDD3 ports: added ACT; removed none
- sheet HDD4 ports: added ACT; removed none
- sheet HDD5 ports: added ACT; removed none
- sheet HDD6 ports: added ACT; removed none
- sheet MCU ports: added ACT_HDD1, ACT_HDD2, ACT_HDD3, ACT_HDD4, ACT_HDD5, ACT_HDD6, MCU_USB_D+, MCU_USB_D-; removed none
- sheet Power ports: added MCU_USB_D+, MCU_USB_D-; removed none
