File: 2-ECAD/hdd.kicad_sch (KiCad schematic)
At the start: 8 parts, among them J13 XUTS-2218-0127, J7 SATA-701-M07S1BR-A

Commit message: production version
Parts:
- removed C17: 100uF, symbol Device:C_Polarized
- removed C23, C35: 0.1uF, symbol Device:C
- removed C29: 47uF, symbol Device:C
- removed D16, D24: D_TVS, symbol Device:D_TVS
- removed J13: XUTS-2218-0127, symbol 0_Connector:XUTS-2218-0127
- removed J7: SATA-701-M07S1BR-A, symbol 0_Connector:SATA-701-M07S1BR-A
- added C401: GRM32ER71A476KE15L, 0_Capacitor:GRM32ER71A476KE15L, symbol 0_Capacitor:GRM32ER71A476KE15L
- added C402, C404: CC0402KRX7R8BB104, 0_Capacitor:C_0402, symbol 0_Capacitor:CC0402KRX7R8BB104
- added C403: UCL1E101MCL1GS, 0_Capacitor:UCL1E101MCL1GS, symbol 0_Capacitor:UCL1E101MCL1GS
- added D401: SMBJ5.0A, 0_Diode:SMBJ5.0A, symbol 0_Diode:SMBJ5.0A
- added D402: SMBJ13A, 0_Diode:SMBJ13A, symbol 0_Diode:SMBJ13A
- added J401: SATA-501-M07S1BY-A, 0_Connector:SATA-501-M07S1BY-A, symbol 0_Connector:SATA-501-M07S1BY-A
- added J402: XUTS-2218-0127, 0_Connector:XUTS-2218-0127, symbol 0_Connector:XUTS-2218-0127
Connections:
- net 12V: now also C403.1, C404.1, D402.1, J402.13 (12V), J402.14 (12V), J402.15 (12V)
- net ACT: now also J402.11 (STA/ACT)
- net GND: now also C401.2, C402.2, C403.2, C404.2, D401.2, D402.2, J401.1 (GND), J401.4 (GND), J401.7 (GND), J401.8 (MP), J401.9 (MP), J402.10 (GND), J402.12 (GND), J402.16 (MP), J402.4 (GND), J402.5 (GND), J402.6 (GND), J402.S1 (GND), J402.S4 (GND), J402.S7 (GND)
- new net +5V: C401.1, C402.1, D401.1, J402.7 (5V), J402.8 (5V), J402.9 (5V)
- new net SATA_A+: J401.2 (A+), J402.S2 (A+)
- new net SATA_A-: J401.3 (A-), J402.S3 (A-)
- new net SATA_B+: J401.6 (B+), J402.S6 (B+)
- new net SATA_B-: J401.5 (B-), J402.S5 (B-)
Other:
- note added: "SATA CONNECTORS"
