File: 2-ECAD/power.kicad_sch (KiCad schematic)
At the start: 39 parts, among them J3 M5082VK-04P, J4 M5082VK-04P, J5 USB4105, Q1 AO3401A, Q2 LMBT3906DW1T1G, Q3 AO3401A, U2 SY8088AAC, U3 SY8088AAC, U4 CN809M

Commit message: production version
Parts:
- removed C10, C14, C7, C8: 10u, symbol Device:C
- removed C11, C13, C5, C9: 0.1u, symbol Device:C
- removed C12, C6: 22p, symbol Device:C
- removed C15: 22uF, symbol Device:C
- removed C16: 0.1uF, symbol Device:C
- removed J3, J4: M5082VK-04P, symbol 0_Connector:M5082VK-04P
- removed J5: USB4105, symbol 0_Connector:USB4105
- removed L1, L2: 2.2u, symbol Device:L
- removed Q1, Q3: AO3401A, symbol 0_Transistor:AO3401A
- removed Q2: LMBT3906DW1T1G, symbol 0_Transistor:LMBT3906DW1T1G
- removed R10, R13: 150k, symbol Device:R
- removed R11, R15, R8: 10k, symbol Device:R
- removed R12, R9: 680k, symbol Device:R
- removed R14: 51k, symbol Device:R
- removed R16: 100k, symbol Device:R
- removed R4, R5: 5.1k, symbol Device:R
- removed R6, R7: 33R, symbol Device:R
- removed U2, U3: SY8088AAC, symbol 0_Converter_DCDC:SY8088AAC
- removed U4: CN809M, symbol 0_Power_Supervisor:CN809M
- added C201: CC0402KRX5R8BB105, 0_Capacitor:C_0402, symbol 0_Capacitor:CC0402KRX5R8BB105
- added C202, C203, C204: EMZR250ARA471MHA0G, 0_Capacitor:EMZR250ARA471MHA0G, symbol 0_Capacitor:EMZR250ARA471MHA0G
- added C205, C209: CC0603KRX5R8BB106, 0_Capacitor:C_0603, symbol 0_Capacitor:CC0603KRX5R8BB106
- added C206, C208, C210, C212: CC0402KRX7R8BB104, 0_Capacitor:C_0402, symbol 0_Capacitor:CC0402KRX7R8BB104
- added C207: CC0402FRNPO9BN220, 0_Capacitor:C_0402, symbol 0_Capacitor:CC0402FRNPO9BN220
- added C211: CC0603MRX5R6BB226, 0_Capacitor:C_0603, symbol 0_Capacitor:CC0603MRX5R6BB226
- added D204: SS34, 0_Diode:SS34, symbol 0_Diode:SS34
- added J201: USB4120, 0_Connector:USB4120, symbol 0_Connector:USB4120
- added J202, J203: 350211-1, 0_Connector:350211-1, symbol 0_Connector:350211-1
- added L201: SRN4018BTA-2R2M, 0_Inductor:SRN4018BTA-2R2M, symbol 0_Inductor:SRN4018BTA-2R2M
- added Q201: AO3401A, 0_Transistor:AO3401A, symbol 0_Transistor:AO3401A
- added R201, R202: RC0402FR-0733RL, 0_Resistor:R_0402, symbol 0_Resistor:RC0402FR-0733RL
- added R203, R204: RC0402FR-075K1L, 0_Resistor:R_0402, symbol 0_Resistor:RC0402FR-075K1L
- added R205: RC0402FR-0710KL, 0_Resistor:R_0402, symbol 0_Resistor:RC0402FR-0710KL
- added R206, R208: RC0402FR-07100KL, 0_Resistor:R_0402, symbol 0_Resistor:RC0402FR-07100KL
- added R207: RC0402FR-0722R1L, 0_Resistor:R_0402, symbol 0_Resistor:RC0402FR-0722R1L
- added U201: SY8088AAC, 0_Converter_DCDC:SY8088AAC, symbol 0_Converter_DCDC:SY8088AAC
- added U202: CN809M, 0_Power_Supervisor:CN809M, symbol 0_Power_Supervisor:CN809M
- D201: renamed from D3; footprint (none) -> 0_Diode:LESD5D5.0CT1G
- D202: renamed from D1; footprint (none) -> 0_Diode:LESD5D5.0CT1G
- D203: renamed from D2; footprint (none) -> 0_Diode:LESD5D5.0CT1G
Connections:
- net GND: now also C201.2, C202.2, C203.2, C204.2, C205.2, C206.2, C208.2, C209.2, C210.2, C211.2, C212.2, J201.1 (MP), J201.2 (MP), J201.3 (MP), J201.4 (MP), J201.A1 (GND), J201.A12 (GND), J201.B1 (GND), J201.B12 (GND), J202.2 (GND), J202.3 (GND), J203.2 (GND), J203.3 (GND), R203.2, R204.2, R207.2, R208.2, U201.2 (GND), U202.1 (GND)
- net MCU_USB_D+: now also R202.2
- net MCU_USB_D-: now also R201.2
- net VBUS: now also C201.1, J201.A4 (VBUS), J201.A9 (VBUS), J201.B4 (VBUS), J201.B9 (VBUS), Q201.3
- net USB_D+: now reaches D203.1
- net USB_D+: now also J201.A7 (Dn1), J201.B7 (Dn2), R202.1
- net USB_D-: now reaches D202.1
- net USB_D-: now also J201.A6 (Dp1), J201.B6 (Dp2), R201.1
- new net: L201.1, U201.3 (LX)
- new net: R205.2, U201.1 (EN)
- new net: Q201.1, R208.1, U202.2 (~{RST})
- new net: J201.B5 (CC2), R203.1
- new net: J201.A5 (CC1), R204.1
- new net: C207.2, R206.2, R207.1, U201.5 (FB)
- new net +12VA: C202.1, J202.1 (12V)
- new net +12VB: C203.1, J203.1 (12V)
- new net +3V3: C207.1, C208.1, C209.1, L201.2, R206.1
- new net +5V: C204.1, C212.1, D204.2, J202.4 (5V), J203.4 (5V), U202.3 (VCC)
- new net VDD: C205.1, C206.1, C210.1, C211.1, D204.1, Q201.2, R205.1, U201.4 (IN)
Other:
- note added: "BUCK CONVERTER"
- note added: "MOLEX POWER IN"
- note added: "POWER PATH"
- note added: "USB-C"
- moved on the sheet: D201, D202, D203
